File: FirstKeyboard/FirstKeyboard.kicad_pcb (KiCad board)
At the start: 2 copper layers, 24 parts, among them J1 USB_B_Mini, SW1 MXSwitch, SW2 MXSwitch, SW3 MXSwitch, SW4 MXSwitch, U1 ATmega32U4-AU, Y1 16MHz

Commit message: Finished Schematic?
Parts:
- added D10: 1N4148W, Diode_SMD:D_SOD-123, F.Cu at (344.2, 70.3)
- added D11: 1N4148W, Diode_SMD:D_SOD-123, F.Cu at (338.5, 70.3)
- added D12: 1N4148W, Diode_SMD:D_SOD-123, F.Cu at (344.2, 67.0)
- added D13: 1N4148W, Diode_SMD:D_SOD-123, F.Cu at (205.8, 214.7)
- added D14: 1N4148W, Diode_SMD:D_SOD-123, F.Cu at (188.6, 208.0)
- added D15: 1N4148W, Diode_SMD:D_SOD-123, F.Cu at (188.6, 214.7)
- added D16: 1N4148W, Diode_SMD:D_SOD-123, F.Cu at (208.2, 211.4)
- added D17: 1N4148W, Diode_SMD:D_SOD-123, F.Cu at (202.4, 211.4)
- added D18: 1N4148W, Diode_SMD:D_SOD-123, F.Cu at (196.7, 211.4)
- added D19: 1N4148W, Diode_SMD:D_SOD-123, F.Cu at (211.6, 208.0)
- added D20: 1N4148W, Diode_SMD:D_SOD-123, F.Cu at (205.8, 208.0)
- added D21: 1N4148W, Diode_SMD:D_SOD-123, F.Cu at (217.3, 204.7)
- added D22: 1N4148W, Diode_SMD:D_SOD-123, F.Cu at (211.6, 204.7)
- added D23: 1N4148W, Diode_SMD:D_SOD-123, F.Cu at (205.8, 204.7)
- added D24: 1N4148W, Diode_SMD:D_SOD-123, F.Cu at (200.1, 208.0)
- added D25: 1N4148W, Diode_SMD:D_SOD-123, F.Cu at (194.3, 204.7)
- added D26: 1N4148W, Diode_SMD:D_SOD-123, F.Cu at (190.9, 211.4)
- added D27: 1N4148W, Diode_SMD:D_SOD-123, F.Cu at (194.3, 214.7)
- added D28: 1N4148W, Diode_SMD:D_SOD-123, F.Cu at (338.5, 67.0)
- added D29: 1N4148W, Diode_SMD:D_SOD-123, F.Cu at (344.2, 63.6)
- added D30: 1N4148W, Diode_SMD:D_SOD-123, F.Cu at (200.1, 204.7)
- added D31: 1N4148W, Diode_SMD:D_SOD-123, F.Cu at (338.5, 63.6)
- added D32: 1N4148W, Diode_SMD:D_SOD-123, F.Cu at (182.8, 214.7)
- added D33: 1N4148W, Diode_SMD:D_SOD-123, F.Cu at (177.1, 214.7)
- added D34: 1N4148W, Diode_SMD:D_SOD-123, F.Cu at (185.2, 211.4)
- added D35: 1N4148W, Diode_SMD:D_SOD-123, F.Cu at (179.4, 211.4)
- added D36: 1N4148W, Diode_SMD:D_SOD-123, F.Cu at (194.3, 208.0)
- added D37: 1N4148W, Diode_SMD:D_SOD-123, F.Cu at (223.1, 204.7)
- added D38: 1N4148W, Diode_SMD:D_SOD-123, F.Cu at (338.5, 83.7)
- added D39: 1N4148W, Diode_SMD:D_SOD-123, F.Cu at (182.8, 208.0)
- added D40: 1N4148W, Diode_SMD:D_SOD-123, F.Cu at (177.1, 208.0)
- added D41: 1N4148W, Diode_SMD:D_SOD-123, F.Cu at (173.7, 211.4)
- added D42: 1N4148W, Diode_SMD:D_SOD-123, F.Cu at (171.3, 214.7)
- added D43: 1N4148W, Diode_SMD:D_SOD-123, F.Cu at (182.8, 204.7)
- added D44: 1N4148W, Diode_SMD:D_SOD-123, F.Cu at (165.6, 214.7)
- added D45: 1N4148W, Diode_SMD:D_SOD-123, F.Cu at (159.8, 214.7)
- added D46: 1N4148W, Diode_SMD:D_SOD-123, F.Cu at (154.1, 214.7)
- added D47: 1N4148W, Diode_SMD:D_SOD-123, F.Cu at (167.9, 211.4)
- added D48: 1N4148W, Diode_SMD:D_SOD-123, F.Cu at (159.8, 204.7)
- added D49: 1N4148W, Diode_SMD:D_SOD-123, F.Cu at (188.6, 204.7)
- added D5: 1N4148W, Diode_SMD:D_SOD-123, F.Cu at (338.5, 80.4)
- added D50: 1N4148W, Diode_SMD:D_SOD-123, F.Cu at (156.4, 211.4)
- added D51: 1N4148W, Diode_SMD:D_SOD-123, F.Cu at (171.3, 208.0)
- added D52: 1N4148W, Diode_SMD:D_SOD-123, F.Cu at (165.6, 208.0)
- added D53: 1N4148W, Diode_SMD:D_SOD-123, F.Cu at (177.1, 204.7)
- added D54: 1N4148W, Diode_SMD:D_SOD-123, F.Cu at (171.3, 204.7)
- added D55: 1N4148W, Diode_SMD:D_SOD-123, F.Cu at (165.6, 204.7)
- added D56: 1N4148W, Diode_SMD:D_SOD-123, F.Cu at (159.8, 208.0)
- added D57: 1N4148W, Diode_SMD:D_SOD-123, F.Cu at (154.1, 208.0)
- added D58: 1N4148W, Diode_SMD:D_SOD-123, F.Cu at (150.7, 211.4)
- added D59: 1N4148W, Diode_SMD:D_SOD-123, F.Cu at (148.3, 214.7)
- added D6: 1N4148W, Diode_SMD:D_SOD-123, F.Cu at (344.2, 77.0)
- added D60: 1N4148W, Diode_SMD:D_SOD-123, F.Cu at (119.5, 214.7)
- added D61: 1N4148W, Diode_SMD:D_SOD-123, F.Cu at (144.9, 211.4)
- added D62: 1N4148W, Diode_SMD:D_SOD-123, F.Cu at (139.2, 211.4)
- added D63: 1N4148W, Diode_SMD:D_SOD-123, F.Cu at (148.3, 208.0)
- added D64: 1N4148W, Diode_SMD:D_SOD-123, F.Cu at (154.1, 204.7)
- added D65: 1N4148W, Diode_SMD:D_SOD-123, F.Cu at (148.3, 204.7)
- added D66: 1N4148W, Diode_SMD:D_SOD-123, F.Cu at (142.6, 208.0)
- added D67: 1N4148W, Diode_SMD:D_SOD-123, F.Cu at (136.8, 214.7)
- added D68: 1N4148W, Diode_SMD:D_SOD-123, F.Cu at (131.1, 214.7)
- added D69: 1N4148W, Diode_SMD:D_SOD-123, F.Cu at (125.3, 214.7)
- added D7: 1N4148W, Diode_SMD:D_SOD-123, F.Cu at (338.5, 77.0)
- added D70: 1N4148W, Diode_SMD:D_SOD-123, F.Cu at (133.4, 211.4)
- added D71: 1N4148W, Diode_SMD:D_SOD-123, F.Cu at (108.0, 214.7)
- added D72: 1N4148W, Diode_SMD:D_SOD-123, F.Cu at (142.6, 214.7)
- added D73: 1N4148W, Diode_SMD:D_SOD-123, F.Cu at (125.3, 208.0)
- added D74: 1N4148W, Diode_SMD:D_SOD-123, F.Cu at (131.1, 204.7)
- added D75: 1N4148W, Diode_SMD:D_SOD-123, F.Cu at (136.8, 204.7)
- added D76: 1N4148W, Diode_SMD:D_SOD-123, F.Cu at (131.1, 208.0)
- added D77: 1N4148W, Diode_SMD:D_SOD-123, F.Cu at (121.9, 211.3)
- added D78: 1N4148W, Diode_SMD:D_SOD-123, F.Cu at (142.6, 204.7)
- added D79: 1N4148W, Diode_SMD:D_SOD-123, F.Cu at (136.8, 208.0)
- added D8: 1N4148W, Diode_SMD:D_SOD-123, F.Cu at (344.2, 73.7)
- added D80: 1N4148W, Diode_SMD:D_SOD-123, F.Cu at (127.7, 211.4)
- added D81: 1N4148W, Diode_SMD:D_SOD-123, F.Cu at (113.8, 214.7)
- added D82: 1N4148W, Diode_SMD:D_SOD-123, F.Cu at (162.2, 211.4)
- added D9: 1N4148W, Diode_SMD:D_SOD-123, F.Cu at (338.5, 73.7)
- added R5: 10k, Resistor_SMD:R_1206_3216Metric_Pad1.42x1.75mm_HandSolder, F.Cu at (114.1, 211.4)
- added SW10: A, acheron_MX:MX100, F.Cu at (244.9, 192.9)
- added SW11: Super, acheron_MX:MX100, F.Cu at (265.1, 172.8)
- added SW12: F2, acheron_MX:MX100, F.Cu at (285.2, 152.6)
- added SW13: Two, acheron_MX:MX100, F.Cu at (265.1, 192.9)
- added SW14: W, acheron_MX:MX100, F.Cu at (184.5, 192.9)
- added SW15: S, acheron_MX:MX100, F.Cu at (265.1, 132.5)
- added SW16: Z, acheron_MX:MX100, F.Cu at (83.7, 192.9)
- added SW17: Alt, acheron_MX:MX100, F.Cu at (184.5, 72.0)
- added SW18: F3, acheron_MX:MX100, F.Cu at (265.1, 92.2)
- added SW19: Three, acheron_MX:MX100, F.Cu at (204.6, 92.2)
- added SW20: E, acheron_MX:MX100, F.Cu at (224.8, 172.8)
- added SW21: D, acheron_MX:MX100, F.Cu at (204.6, 192.9)
- added SW22: X, acheron_MX:MX100, F.Cu at (305.4, 72.0)
- added SW23: F4, acheron_MX:MX100, F.Cu at (285.2, 92.2)
- added SW24: Four, acheron_MX:MX100, F.Cu at (265.1, 112.3)
- added SW25: R, acheron_MX:MX100, F.Cu at (244.9, 132.5)
- added SW26: F, acheron_MX:MX100, F.Cu at (224.8, 152.6)
- added SW27: C, acheron_MX:MX100, F.Cu at (204.6, 172.8)
- added SW28: F5, acheron_MX:MX100, F.Cu at (184.5, 152.6)
- added SW29: Five, acheron_MX:MX100, F.Cu at (285.2, 72.0)
- added SW30: T, acheron_MX:MX100, F.Cu at (244.9, 152.6)
- added SW31: G, acheron_MX:MX100, F.Cu at (244.9, 112.3)
- added SW32: V, acheron_MX:MX100, F.Cu at (224.8, 132.5)
- added SW33: F6, acheron_MX:MX100, F.Cu at (204.6, 152.6)
- added SW34: Six, acheron_MX:MX100, F.Cu at (184.5, 172.8)
- added SW35: Y, acheron_MX:MX100, F.Cu at (164.3, 192.9)
- added SW36: H, acheron_MX:MX100, F.Cu at (265.1, 72.0)
- added SW37: B, acheron_MX:MX100, F.Cu at (244.9, 92.2)
- added SW38: Space, acheron_MX:MX100, F.Cu at (224.8, 112.3)
- added SW39: F7, acheron_MX:MX100, F.Cu at (204.6, 132.5)
- added SW40: Seven, acheron_MX:MX100, F.Cu at (325.5, 112.3)
- added SW41: U, acheron_MX:MX100, F.Cu at (305.4, 92.2)
- added SW42: J, acheron_MX:MX100, F.Cu at (144.2, 192.9)
- added SW43: N, acheron_MX:MX100, F.Cu at (244.9, 72.0)
- added SW44: F8, acheron_MX:MX100, F.Cu at (224.8, 92.2)
- added SW45: Eight, acheron_MX:MX100, F.Cu at (204.6, 112.3)
- added SW46: I, acheron_MX:MX100, F.Cu at (184.5, 132.5)
- added SW47: K, acheron_MX:MX100, F.Cu at (164.3, 152.6)
- added SW48: M, acheron_MX:MX100, F.Cu at (144.2, 172.8)
- added SW49: F9, acheron_MX:MX100, F.Cu at (124.0, 192.9)
- added SW5: Shift, acheron_MX:MX100, F.Cu at (224.8, 192.9)
- added SW50: Nine, acheron_MX:MX100, F.Cu at (224.8, 72.0)
- added SW51: O, acheron_MX:MX100, F.Cu at (103.9, 172.8)
- added SW52: L, acheron_MX:MX100, F.Cu at (164.3, 172.8)
- added SW53: <, acheron_MX:MX100, F.Cu at (184.5, 112.3)
- added SW54: F10, acheron_MX:MX100, F.Cu at (164.3, 132.5)
- added SW55: Zero, acheron_MX:MX100, F.Cu at (144.2, 152.6)
- added SW56: P, acheron_MX:MX100, F.Cu at (124.0, 172.8)
- added SW57: Colon, acheron_MX:MX100, F.Cu at (103.9, 192.9)
- added SW58: >, acheron_MX:MX100, F.Cu at (204.6, 72.0)
- added SW59: Alt, acheron_MX:MX100, F.Cu at (184.5, 92.2)
- added SW6: Ctrl, acheron_MX:MX100, F.Cu at (325.5, 72.0)
- added SW60: F11, acheron_MX:MX100, F.Cu at (164.3, 112.3)
- added SW61: Minus, acheron_MX:MX100, F.Cu at (144.2, 132.5)
- added SW62: [, acheron_MX:MX100, F.Cu at (124.0, 152.6)
- added SW63: Quote, acheron_MX:MX100, F.Cu at (103.9, 112.3)
- added SW64: ?, acheron_MX:MX100, F.Cu at (144.2, 112.3)
- added SW65: Fn, acheron_MX:MX100, F.Cu at (124.0, 132.5)
- added SW66: F12, acheron_MX:MX100, F.Cu at (103.9, 152.6)
- added SW67: Plus, acheron_MX:MX100, F.Cu at (83.7, 172.8)
- added SW68: ], acheron_MX:MX100, F.Cu at (164.3, 72.0)
- added SW69: Shift, acheron_MX:MX100, F.Cu at (144.2, 92.2)
- added SW7: F1, acheron_MX:MX100, F.Cu at (305.4, 132.5)
- added SW70: Left, acheron_MX:MX100, F.Cu at (124.0, 112.3)
- added SW71: Home, acheron_MX:MX100, F.Cu at (83.7, 72.0)
- added SW72: BkSpc, acheron_MX:MX100, F.Cu at (83.7, 152.6)
- added SW73: \, acheron_MX:MX100, F.Cu at (144.2, 72.0)
- added SW74: Enter, acheron_MX:MX100, F.Cu at (124.0, 92.2)
- added SW75: Up, acheron_MX:MX100, F.Cu at (164.3, 92.2)
- added SW76: Down, acheron_MX:MX100, F.Cu at (83.7, 132.5)
- added SW77: End, acheron_MX:MX100, F.Cu at (124.0, 72.0)
- added SW78: Delete, acheron_MX:MX100, F.Cu at (103.9, 92.2)
- added SW79: PgUp, acheron_MX:MX100, F.Cu at (83.7, 112.3)
- added SW8: One, acheron_MX:MX100, F.Cu at (285.2, 112.3)
- added SW80: PgDn, acheron_MX:MX100, F.Cu at (103.9, 72.0)
- added SW81: Right, acheron_MX:MX100, F.Cu at (83.7, 92.2)
- added SW82: Ins, acheron_MX:MX100, F.Cu at (103.9, 132.5)
- added SW9: Q, acheron_MX:MX100, F.Cu at (325.5, 92.2)
- C1: value 100n -> 1uF
- C4: value 1uF -> 100n
- D1, D2, D3, D4: value D_Small -> 1N4148W
- R1: value 10k -> 1k
- R4: value 10k -> 330
- SW1: value MXSwitch -> Esc
- SW2: value MXSwitch -> Tilde
- SW3: value MXSwitch -> Tab
- SW4: value MXSwitch -> CapsL
- moved D2 229.2 mm to (344.2, 80.4)
- moved SW1 215.0 mm to (305.4, 112.3)
- moved SW2 195.6 mm to (285.2, 132.5)
- moved D1 194.7 mm to (338.5, 87.1)
- moved D4 177.6 mm to (211.6, 214.7)
- moved SW3 176.6 mm to (265.1, 152.6)
- moved C3 174.7 mm to (235.8, 204.5)
- moved C2 172.0 mm to (231.1, 207.4)
- moved J1 168.3 mm to (93.7, 205.9)
- moved U1 168.3 mm to (80.9, 210.2)
- moved C7 167.3 mm to (216.8, 207.8)
- moved C6 166.0 mm to (221.6, 207.8)
- moved C8 164.8 mm to (213.4, 211.2)
- moved C4 163.7 mm to (231.1, 204.5)
- moved C5 161.7 mm to (226.3, 207.8)
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Connections:
- C1 pad 1: GND -> Net-(C1-Pad1)
- C1 pad 2: RST -> GND
- C2 pad 1: Net-(C2-Pad1) -> GND
- C2 pad 2: GND -> Net-(C2-Pad2)
- C3 pad 1: GND -> Net-(C3-Pad1)
- C3 pad 2: Net-(C3-Pad2) -> GND
- C4 pad 2: GND -> RST
- D1 pad 1: Col1 -> Row1
- D2 pad 1: Col2 -> Row2
- D3 pad 1: Col1 -> Row3
- D4 pad 1: Col2 -> Row4
- R1 pad 1: RST -> GND
- R1 pad 2: +5V -> Net-(R1-Pad2)
- R2 pad 1: Net-(R2-Pad1) -> Net-(J1-Pad2)
- R2 pad 2: Net-(J1-Pad3) -> Net-(R2-Pad2)
- R3 pad 1: Net-(J1-Pad2) -> Net-(R3-Pad1)
- R3 pad 2: Net-(R3-Pad2) -> Net-(J1-Pad3)
- R4 pad 1: GND -> Net-(C4-Pad1)
- R4 pad 2: Net-(R4-Pad2) -> GND
- SW1 pad 1: Row1 -> Col1
- SW2 pad 1: Row1 -> Col1
- SW3 pad 1: Row2 -> Col1
- SW4 pad 1: Row2 -> Col1
- SWP1 pad 1: GND -> Net-(C4-Pad1)
- U1 pad 16: Net-(C3-Pad2) -> Net-(C2-Pad2)
- U1 pad 17: Net-(C2-Pad1) -> Net-(C3-Pad1)
- U1 pad 3: Net-(R3-Pad2) -> Net-(R2-Pad2)
- U1 pad 33: Net-(R4-Pad2) -> Net-(R1-Pad2)
- U1 pad 4: Net-(R2-Pad1) -> Net-(R3-Pad1)
- U1 pad 6: Net-(C4-Pad1) -> Net-(C1-Pad1)
- Y1 pad 1: Net-(C3-Pad2) -> Net-(C2-Pad2)
- Y1 pad 2: Net-(C2-Pad1) -> Net-(C3-Pad1)

Commit message: Removed the "INS" key
Parts:
- removed D82: 1N4148W, Diode_SMD:D_SOD-123
- removed SW82: Ins, acheron_MX:MX100
- moved D31 224.7 mm to (166.0, 207.6)
- moved D29 216.0 mm to (177.5, 200.9)
- moved D6 209.5 mm to (183.0, 210.9)
- moved D28 205.0 mm to (183.2, 200.9)
- moved D8 205.0 mm to (189.0, 207.6)
- moved D9 205.0 mm to (183.2, 207.6)
- moved D3 201.2 mm to (332.3, 63.2)
- moved D5 198.6 mm to (188.8, 210.9)
- moved SW41 198.4 mm to (132.3, 189.1)
- moved D18 197.1 mm to (326.6, 63.2)
- moved D10 196.4 mm to (200.5, 204.2)
- moved D11 196.4 mm to (194.7, 204.2)
- moved D12 196.4 mm to (200.5, 200.9)
- moved D7 194.2 mm to (194.7, 207.6)
- moved D38 192.1 mm to (194.5, 210.9)
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
Commit message: Small update to Aly keys
Parts:
- SW17: value Alt -> LAlt
- SW59: value Alt -> RAlt
- moved C4 10.0 mm to (335.6, 79.1)
- moved SW1 10.0 mm to (282.8, 131.8)
- moved SW14 10.0 mm to (282.8, 71.4)
- moved SW6 10.0 mm to (282.8, 152.0)
- moved U1 10.0 mm to (259.8, 189.4)
- moved C3 10.0 mm to (335.6, 82.1)
- moved C5 10.0 mm to (340.3, 76.2)
- moved C6 10.0 mm to (335.6, 76.2)
- moved D1 10.0 mm to (341.8, 69.7)
- moved D13 10.0 mm to (336.1, 69.7)
- moved D18 10.0 mm to (336.1, 66.3)
- moved D19 10.0 mm to (341.8, 63.0)
- moved D21 10.0 mm to (336.1, 63.0)
- moved D3 10.0 mm to (341.8, 66.3)
- moved D37 10.0 mm to (341.8, 73.0)
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
Commit message: Updating the keyboard layout
Parts:
- C1, C2, C3, C4, C5, C6, C7, C8, D1, D10, D11, D12, D13, D14, D15, D16, D17, D18, D19, D2, D20, D21, D22, D23, D24, D25, D26, D27, D28, D29, D3, D30, D31, D32, D33, D34, D35, D36, D37, D38, D39, D4, D40, D41, D42, D43, D44, D45, D46, D47, D48, D49, D5, D50, D51, D52, D53, D54, D55, D56, D57, D58, D59, D6, D60, D61, D62, D63, D64, D65, D66, D67, D68, D69, D7, D70, D71, D72, D73, D74, D75, D76, D77, D78, D79, D8, D80, D81, D9, J1, R1, R2, R3, R4, R5, SW1, SW10, SW12, SW13, SW14, SW15, SW16, SW18, SW19, SW2, SW20, SW21, SW22, SW23, SW24, SW25, SW26, SW28, SW29, SW30, SW31, SW32, SW33, SW34, SW35, SW36, SW37, SW39, SW40, SW41, SW42, SW43, SW44, SW45, SW46, SW47, SW48, SW49, SW50, SW51, SW52, SW53, SW54, SW55, SW56, SW57, SW58, SW60, SW61, SW62, SW63, SW64, SW66, SW67, SW68, SW7, SW70, SW71, SW75, SW76, SW77, SW78, SW79, SW8, SW80, SW81, SW9, SWP1, U1, Y1: moved to B.Cu
- SW11: value Super -> Super_125; footprint acheron_MX:MX100 -> acheron_MX:MX125; moved to B.Cu
- SW17: value LAlt -> LAlt_125; footprint acheron_MX:MX100 -> acheron_MX:MX125; moved to B.Cu
- SW3: value Tab -> Tab_125; footprint acheron_MX:MX100 -> acheron_MX:MX125; moved to B.Cu
- SW38: value Space -> Space_625; footprint acheron_MX:MX100 -> acheron_MX:MX625; moved to B.Cu
- SW4: value CapsL -> Caps_175; footprint acheron_MX:MX100 -> acheron_MX:MX175; moved to B.Cu
- SW5: value Shift -> Shift_2.25; footprint acheron_MX:MX100 -> acheron_MX:MX225; moved to B.Cu
- SW59: value RAlt -> RAlt_125; footprint acheron_MX:MX100 -> acheron_MX:MX125; moved to B.Cu
- SW6: value Ctrl -> LCtrl_125; footprint acheron_MX:MX100 -> acheron_MX:MX125; moved to B.Cu
- SW65: value Fn -> Fn_150; footprint acheron_MX:MX100 -> acheron_MX:MX150; moved to B.Cu
- SW69: value Shift -> Shift_175; footprint acheron_MX:MX100 -> acheron_MX:MX175; moved to B.Cu
- SW72: value BkSpc -> BkSpc_2; footprint acheron_MX:MX100 -> acheron_MX:MX200; moved to B.Cu
- SW73: value \ -> \_150; footprint acheron_MX:MX100 -> acheron_MX:MX150; moved to B.Cu
- SW74: value Enter -> Enter_225; footprint acheron_MX:MX100 -> acheron_MX:MX225; moved to B.Cu
- moved SW16 711.2 mm to (790.7, 141.6), turned to 180 degrees
- moved SW51 687.9 mm to (783.4, 40.9), turned to 180 degrees
- moved SW46 641.1 mm to (796.6, 61.0), turned to 180 degrees
- moved SW41 619.8 mm to (736.9, 18.8), turned to 180 degrees
- moved SW37 609.4 mm to (810.8, 101.3), turned to 180 degrees
- moved SW26 584.8 mm to (756.3, 81.2), turned to 180 degrees
- moved SW32 584.8 mm to (756.3, 61.0), turned to 180 degrees
- moved SW52 571.9 mm to (742.7, -1.32), turned to 180 degrees
- moved SW30 569.1 mm to (790.7, 101.3), turned to 180 degrees
- moved SW27 556.2 mm to (696.6, 18.8)
- moved SW25 545.7 mm to (736.1, 59.1), turned to 180 degrees
- moved SW31 532.8 mm to (722.9, 39.0), turned to 180 degrees
- moved SW15 528.9 mm to (770.5, 121.5), turned to 180 degrees
- moved SW22 508.0 mm to (770.5, 101.3), turned to 180 degrees
- moved SW35 503.3 mm to (743.1, 39.0), turned to 180 degrees
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
Commit message: Keys are in place. Next diodes?
Parts:
- SW3: value Tab_125 -> Tab_150; footprint acheron_MX:MX125 -> acheron_MX:MX150
- moved SW16 696.2 mm to (95.2, 109.5)
- moved SW15 666.5 mm to (104.8, 90.5)
- moved SW22 656.3 mm to (114.3, 109.5)
- moved SW14 651.1 mm to (100.0, 71.4)
- moved SW37 639.4 mm to (171.4, 109.5)
- moved SW30 634.2 mm to (157.2, 71.4)
- moved SW26 613.5 mm to (142.9, 90.5)
- moved SW10 610.9 mm to (85.7, 90.5)
- moved SW32 605.8 mm to (152.4, 109.5)
- moved SW25 598.1 mm to (138.1, 71.4)
- moved SW46 582.3 mm to (214.3, 71.4)
- moved SW21 581.2 mm to (123.8, 90.5)
- moved SW27 570.5 mm to (133.3, 109.5)
- moved SW35 567.8 mm to (176.2, 71.4)
- moved SW31 563.4 mm to (161.9, 90.5)
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
Commit message: Re-added pcb cut edge
Other:
- board outline added: 309.6 x 119.1 mm
Changed lines of the file:
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@@
   (general
     (thickness 1.6)
-    (drawings 0)
+    (drawings 8)
     (tracks 0)
     (zones 0)
@@
     )
   )
+  (gr_arc (start 345.28125 26.19375) (end 350.04375 26.19375) (angle -90) (layer Edge.Cuts) (width 0.05))
+  (gr_arc (start 345.28125 135.73125) (end 345.28125 140.49375) (angle -90) (layer Edge.Cuts) (width 0.05))
+  (gr_arc (start 45.24375 135.73125) (end 40.48125 135.73125) (angle -90) (layer Edge.Cuts) (width 0.05))
+  (gr_arc (start 45.24375 26.19375) (end 45.24375 21.43125) (angle -90) (layer Edge.Cuts) (width 0.05))
+  (gr_line (start 345.28125 21.43125) (end 45.24375 21.43125) (layer Edge.Cuts) (width 0.05))
+  (gr_line (start 350.04375 135.73125) (end 350.04375 26.19375) (layer Edge.Cuts) (width 0.05))
+  (gr_line (start 45.24375 140.49375) (end 345.28125 140.49375) (layer Edge.Cuts) (width 0.05))
+  (gr_line (start 40.48125 26.19375) (end 40.48125 135.73125) (layer Edge.Cuts) (width 0.05))
 )

Commit message: updated assigned footprints and pcb from Schema
Parts:
- J1: moved to F.Cu
- SW1, SW10, SW12, SW13, SW14, SW15, SW16, SW18, SW19, SW2, SW20, SW21, SW22, SW23, SW24, SW25, SW26, SW27, SW28, SW29, SW30, SW31, SW32, SW33, SW34, SW35, SW36, SW37, SW39, SW40, SW41, SW42, SW43, SW44, SW45, SW46, SW47, SW48, SW49, SW50, SW51, SW52, SW53, SW54, SW55, SW56, SW57, SW58, SW60, SW61, SW62, SW63, SW64, SW66, SW67, SW68, SW7, SW70, SW71, SW75, SW76, SW77, SW78, SW79, SW8, SW80, SW81, SW9: footprint acheron_MX:MX100 -> acheron_MX:MX100P
- SW11, SW17, SW59, SW6: footprint acheron_MX:MX125 -> acheron_MX:MX125P
- SW3, SW65, SW73: footprint acheron_MX:MX150 -> acheron_MX:MX150P
- SW38: footprint acheron_MX:MX625 -> acheron_MX:MX625P
- SW4, SW69: footprint acheron_MX:MX175 -> acheron_MX:MX175P
- SW5, SW74: footprint acheron_MX:MX225 -> acheron_MX:MX225P
- SW72: footprint acheron_MX:MX200 -> acheron_MX:MX200P
- turned J1 to 180 degrees
