File: FirstKeyboard/FirstKeyboard.sch (KiCad schematic (older format))
At the start: 179 parts, among them J1 USB_B_Mini, SW1 Esc, SW10 A, SW11 Super, SW12 F2, SW13 Two, SW14 W, SW15 S, SW16 Z, SW17 LAlt, SW18 F3, SW19 Three, SW2 Tilde, SW20 E, SW21 D, SW22 X, SW23 F4, SW24 Four, SW25 R, SW26 F, SW27 C, SW28 F5, SW29 Five, SW3 Tab, SW30 T, SW31 G, SW32 V, SW33 F6, SW34 Six, SW35 Y, SW36 H, SW37 B, SW38 Space, SW39 F7, SW4 CapsL, SW40 Seven, SW41 U, SW42 J, SW43 N, SW44 F8, SW45 Eight, SW46 I, SW47 K, SW48 M, SW49 F9, SW5 Shift, SW50 Nine, SW51 O, SW52 L, SW53 <, SW54 F10, SW55 Zero, SW56 P, SW57 Colon, SW58 >, SW59 RAlt, SW6 Ctrl, SW60 F11, SW61 Minus, SW62 [, SW63 Quote, SW64 ?, SW65 Fn, SW66 F12, SW67 Plus, SW68 ], SW69 Shift, SW7 F1, SW70 Left, SW71 Home, SW72 BkSpc, SW73 \\, SW74 Enter, SW75 Up, SW76 Down, SW77 End, SW78 Delete, SW79 PgUp, SW8 One, SW80 PgDn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

Commit message: Updating the keyboard layout
Parts:
- SW11: value Super -> Super_125; footprint acheron_MX:MX100 -> acheron_MX:MX125
- SW17: value LAlt -> LAlt_125; footprint acheron_MX:MX100 -> acheron_MX:MX125
- SW3: value Tab -> Tab_125; footprint acheron_MX:MX100 -> acheron_MX:MX125
- SW38: value Space -> Space_625; footprint acheron_MX:MX100 -> acheron_MX:MX625
- SW4: value CapsL -> Caps_175; footprint acheron_MX:MX100 -> acheron_MX:MX175
- SW5: value Shift -> Shift_2.25; footprint acheron_MX:MX100 -> acheron_MX:MX225
- SW59: value RAlt -> RAlt_125; footprint acheron_MX:MX100 -> acheron_MX:MX125
- SW6: value Ctrl -> LCtrl_125; footprint acheron_MX:MX100 -> acheron_MX:MX125
- SW65: value Fn -> Fn_150; footprint acheron_MX:MX100 -> acheron_MX:MX150
- SW69: value Shift -> Shift_175; footprint acheron_MX:MX100 -> acheron_MX:MX175
- SW72: value BkSpc -> BkSpc_2; footprint acheron_MX:MX100 -> acheron_MX:MX200
- SW73: value \\ -> \\_150; footprint acheron_MX:MX100 -> acheron_MX:MX150
- SW74: value Enter -> Enter_225; footprint acheron_MX:MX100 -> acheron_MX:MX225
Changed lines of the file:
@@
 P 5150 3650
 F 0 "SW3" H 5075 3725 50  0000 L CNN
-F 1 "Tab" H 5025 3625 79  0000 L CNN
-F 2 "acheron_MX:MX100" H 5150 3650 50  0001 C CNN
+F 1 "Tab_125" H 4900 3600 79  0000 L CNN
+F 2 "acheron_MX:MX125" H 5150 3650 50  0001 C CNN
 F 3 "" H 5150 3650 50  0001 C CNN
 	1    5150 3650
@@
 P 5150 4575
 F 0 "SW4" H 5075 4650 50  0000 L CNN
-F 1 "CapsL" H 4975 4550 79  0000 L CNN
-F 2 "acheron_MX:MX100" H 5150 4575 50  0001 C CNN
+F 1 "Caps_175" H 4925 4525 59  0000 L CNN
+F 2 "acheron_MX:MX175" H 5150 4575 50  0001 C CNN
 F 3 "" H 5150 4575 50  0001 C CNN
 	1    5150 4575
@@
 P 5150 5500
 F 0 "SW5" H 5075 5575 50  0000 L CNN
-F 1 "Shift" H 5000 5475 79  0000 L CNN
-F 2 "acheron_MX:MX100" H 5150 5500 50  0001 C CNN
+F 1 "Shift_2.25" H 4925 5475 59  0000 L CNN
+F 2 "acheron_MX:MX225" H 5150 5500 50  0001 C CNN
 F 3 "" H 5150 5500 50  0001 C CNN
 	1    5150 5500
@@
 	4525 4900 5150 4900
 $Comp
-L acheronSymbols:MXSwitch SW6
-U 1 1 5E118D86
-P 5150 6425
-F 0 "SW6" H 5075 6500 50  0000 L CNN
-F 1 "Ctrl" H 5025 6400 79  0000 L CNN
-F 2 "acheron_MX:MX100" H 5150 6425 50  0001 C CNN
-F 3 "" H 5150 6425 50  0001 C CNN
-	1    5150 6425
-	1    0    0    -1
-$EndComp
-$Comp
 L Device:D_Small D6
 U 1 1 5E118D8C
@@
 P 5875 6425
 F 0 "SW11" H 5800 6500 50  0000 L CNN
-F 1 "Super" H 5725 6400 79  0000 L CNN
-F 2 "acheron_MX:MX100" H 5875 6425 50  0001 C CNN
+F 1 "Super_125" H 5650 6375 59  0000 L CNN
+F 2 "acheron_MX:MX125" H 5875 6425 50  0001 C CNN
 F 3 "" H 5875 6425 50  0001 C CNN
 	1    5875 6425
@@
 P 14875 3650
 F 0 "SW73" H 14800 3725 50  0000 L CNN
-F 1 "\\" H 14850 3600 79  0000 L CNN
-F 2 "acheron_MX:MX100" H 14875 3650 50  0001 C CNN
+F 1 "\\_150" H 14725 3600 79  0000 L CNN
+F 2 "acheron_MX:MX150" H 14875 3650 50  0001 C CNN
 F 3 "" H 14875 3650 50  0001 C CNN
 	1    14875 3650
@@
 P 14875 5500
 F 0 "SW75" H 14800 5575 50  0000 L CNN
-F 1 "Up" H 14750 5500 79  0000 L CNN
+F 1 "Up" H 14800 5475 79  0000 L CNN
 F 2 "acheron_MX:MX100" H 14875 5500 50  0001 C CNN
 F 3 "" H 14875 5500 50  0001 C CNN
@@
 P 14125 5500
 F 0 "SW69" H 14050 5575 50  0000 L CNN
-F 1 "Shift" H 14000 5500 79  0000 L CNN
-F 2 "acheron_MX:MX100" H 14125 5500 50  0001 C CNN
+F 1 "Shift_175" H 13900 5450 59  0000 L CNN
+F 2 "acheron_MX:MX175" H 14125 5500 50  0001 C CNN
 F 3 "" H 14125 5500 50  0001 C CNN
 	1    14125 5500
@@
 P 6625 6425
 F 0 "SW17" H 6550 6500 50  0000 L CNN
-F 1 "LAlt" H 6525 6400 79  0000 L CNN
-F 2 "acheron_MX:MX100" H 6625 6425 50  0001 C CNN
+F 1 "LAlt_125" H 6425 6375 59  0000 L CNN
+F 2 "acheron_MX:MX125" H 6625 6425 50  0001 C CNN
 F 3 "" H 6625 6425 50  0001 C CNN
 	1    6625 6425
@@
 P 13375 6425
 F 0 "SW65" H 13300 6500 50  0000 L CNN
-F 1 "Fn" H 13300 6400 79  0000 L CNN
-F 2 "acheron_MX:MX100" H 13375 6425 50  0001 C CNN
+F 1 "Fn_150" H 13175 6375 79  0000 L CNN
+F 2 "acheron_MX:MX150" H 13375 6425 50  0001 C CNN
 F 3 "" H 13375 6425 50  0001 C CNN
 	1    13375 6425
@@
 P 9625 6425
 F 0 "SW38" H 9550 6500 50  0000 L CNN
-F 1 "Space" H 9450 6400 79  0000 L CNN
-F 2 "acheron_MX:MX100" H 9625 6425 50  0001 C CNN
+F 1 "Space_625" H 9375 6375 59  0000 L CNN
+F 2 "acheron_MX:MX625" H 9625 6425 50  0001 C CNN
 F 3 "" H 9625 6425 50  0001 C CNN
 	1    9625 6425
@@
 P 15625 6425
 F 0 "SW81" H 15550 6500 50  0000 L CNN
-F 1 "Right" H 15500 6425 79  0000 L CNN
+F 1 "Right" H 15500 6400 79  0000 L CNN
 F 2 "acheron_MX:MX100" H 15625 6425 50  0001 C CNN
 F 3 "" H 15625 6425 50  0001 C CNN
@@
 P 14875 6425
 F 0 "SW76" H 14800 6500 50  0000 L CNN
-F 1 "Down" H 14750 6425 79  0000 L CNN
+F 1 "Down" H 14750 6400 79  0000 L CNN
 F 2 "acheron_MX:MX100" H 14875 6425 50  0001 C CNN
 F 3 "" H 14875 6425 50  0001 C CNN
@@
 P 14125 6425
 F 0 "SW70" H 14050 6500 50  0000 L CNN
-F 1 "Left" H 14000 6425 79  0000 L CNN
+F 1 "Left" H 14000 6400 79  0000 L CNN
 F 2 "acheron_MX:MX100" H 14125 6425 50  0001 C CNN
 F 3 "" H 14125 6425 50  0001 C CNN
@@
 P 14875 2725
 F 0 "SW72" H 14800 2800 50  0000 L CNN
-F 1 "BkSpc" H 14725 2700 79  0000 L CNN
-F 2 "acheron_MX:MX100" H 14875 2725 50  0001 C CNN
+F 1 "BkSpc_2" H 14625 2700 79  0000 L CNN
+F 2 "acheron_MX:MX200" H 14875 2725 50  0001 C CNN
 F 3 "" H 14875 2725 50  0001 C CNN
 	1    14875 2725
@@
 P 12625 6425
 F 0 "SW59" H 12550 6500 50  0000 L CNN
-F 1 "RAlt" H 12525 6400 79  0000 L CNN
-F 2 "acheron_MX:MX100" H 12625 6425 50  0001 C CNN
+F 1 "RAlt_125" H 12425 6375 59  0000 L CNN
+F 2 "acheron_MX:MX125" H 12625 6425 50  0001 C CNN
 F 3 "" H 12625 6425 50  0001 C CNN
 	1    12625 6425
@@
 P 14875 4575
 F 0 "SW74" H 14800 4650 50  0000 L CNN
-F 1 "Enter" H 14725 4550 79  0000 L CNN
-F 2 "acheron_MX:MX100" H 14875 4575 50  0001 C CNN
+F 1 "Enter_225" H 14650 4550 59  0000 L CNN
+F 2 "acheron_MX:MX225" H 14875 4575 50  0001 C CNN
 F 3 "" H 14875 4575 50  0001 C CNN
 	1    14875 4575
@@
 	1    0    0    -1
 $EndComp
+$Comp
+L acheronSymbols:MXSwitch SW6
+U 1 1 5E118D86
+P 5150 6425
+F 0 "SW6" H 5075 6500 50  0000 L CNN
+F 1 "LCtrl_125" H 4950 6375 59  0000 L CNN
+F 2 "acheron_MX:MX125" H 5150 6425 50  0001 C CNN
+F 3 "" H 5150 6425 50  0001 C CNN
+	1    5150 6425
+	1    0    0    -1
+$EndComp

Commit message: Keys are in place. Next diodes?
Parts:
- SW3: value Tab_125 -> Tab_150; footprint acheron_MX:MX125 -> acheron_MX:MX150
Changed lines of the file:
@@
 P 5150 3650
 F 0 "SW3" H 5075 3725 50  0000 L CNN
-F 1 "Tab_125" H 4900 3600 79  0000 L CNN
-F 2 "acheron_MX:MX125" H 5150 3650 50  0001 C CNN
+F 1 "Tab_150" H 4900 3600 79  0000 L CNN
+F 2 "acheron_MX:MX150" H 5150 3650 50  0001 C CNN
 F 3 "" H 5150 3650 50  0001 C CNN
 	1    5150 3650

Commit message: updated assigned footprints and pcb from Schema
Parts:
- SW1, SW10, SW12, SW13, SW14, SW15, SW16, SW18, SW19, SW2, SW20, SW21, SW22, SW23, SW24, SW25, SW26, SW27, SW28, SW29, SW30, SW31, SW32, SW33, SW34, SW35, SW36, SW37, SW39, SW40, SW41, SW42, SW43, SW44, SW45, SW46, SW47, SW48, SW49, SW50, SW51, SW52, SW53, SW54, SW55, SW56, SW57, SW58, SW60, SW61, SW62, SW63, SW64, SW66, SW67, SW68, SW7, SW70, SW71, SW75, SW76, SW77, SW78, SW79, SW8, SW80, SW81, SW9: footprint acheron_MX:MX100 -> acheron_MX:MX100P
- SW11, SW17, SW59, SW6: footprint acheron_MX:MX125 -> acheron_MX:MX125P
- SW3, SW65, SW73: footprint acheron_MX:MX150 -> acheron_MX:MX150P
- SW38: footprint acheron_MX:MX625 -> acheron_MX:MX625P
- SW4, SW69: footprint acheron_MX:MX175 -> acheron_MX:MX175P
- SW5, SW74: footprint acheron_MX:MX225 -> acheron_MX:MX225P
- SW72: footprint acheron_MX:MX200 -> acheron_MX:MX200P
